File: KiCAD/SatFinder/SatFinder.kicad_pcb (KiCad board)
At the start: 2 copper layers, 75.6 x 52.1 mm, 12 parts, among them J1 GY-271, J2 GY-521, J3 D24V10F5, J4 DRV8871, J5 Power, J6 Coax, U1 WeMos_D1_mini

Commit message: Version 1.1
Parts:
- J2: footprint Connector_Wago:Wago_734-134_1x04_P3.50mm_Vertical -> TerminalBlock:TerminalBlock_bornier-4_P5.08mm
- J5, J6: footprint Connector_Wago:Wago_734-132_1x02_P3.50mm_Vertical -> TerminalBlock:TerminalBlock_bornier-2_P5.08mm
- moved J2 3.47 mm to (141.0, 83.2)
- moved J6 2.54 mm to (141.0, 71.1)
- moved J5 1.27 mm to (141.0, 105.4)
Routing:
- net GND: track 143.4 -> 146.0 mm
- net Net-(J1-Pad1): track 121.0 -> 119.6 mm
- net Net-(C1-Pad2): track 44.0 -> 44.7 mm
- net Net-(J1-Pad4): track 96.6 -> 96.1 mm
Other:
- board text added: "+"
- board text added: "-"
- board text added: "SatFinder 1.1"
