File: KiCAD/SatFinder/SatFinder.sch (KiCad schematic (older format))
At the start: 12 parts, among them J1 GY-271, J2 GY-521, J3 D24V10F5, J4 DRV8871, J5 Power, J6 Coax, U1 WeMos_D1_mini

Commit message: Version 1.1
Parts:
- J2: footprint Connector_Wago:Wago_734-134_1x04_P3.50mm_Vertical -> TerminalBlock:TerminalBlock_bornier-4_P5.08mm
- J5, J6: footprint Connector_Wago:Wago_734-132_1x02_P3.50mm_Vertical -> TerminalBlock:TerminalBlock_bornier-2_P5.08mm
Connections:
- wire segments 72 -> 75
Changed lines of the file:
@@
 	3700 2400 5500 2400
-Wire Wire Line
-	3800 2050 3800 2500
 Wire Wire Line
 	2400 2600 3900 2600
@@
 F 0 "J5" H 1418 4817 50  0000 C CNN
 F 1 "Power" H 1418 4726 50  0000 C CNN
-F 2 "Connector_Wago:Wago_734-132_1x02_P3.50mm_Vertical" H 1500 4600 50  0001 C CNN
+F 2 "TerminalBlock:TerminalBlock_bornier-2_P5.08mm" H 1500 4600 50  0001 C CNN
 F 3 "~" H 1500 4600 50  0001 C CNN
 	1    1500 4600
@@
 F 0 "J2" V 3764 1562 50  0000 R CNN
 F 1 "GY-521" V 3673 1562 50  0000 R CNN
-F 2 "Connector_Wago:Wago_734-134_1x04_P3.50mm_Vertical" H 3800 1850 50  0001 C CNN
+F 2 "TerminalBlock:TerminalBlock_bornier-4_P5.08mm" H 3800 1850 50  0001 C CNN
 F 3 "~" H 3800 1850 50  0001 C CNN
 	1    3800 1850
@@
 F 0 "J6" H 1418 7017 50  0000 C CNN
 F 1 "Coax" H 1418 6926 50  0000 C CNN
-F 2 "Connector_Wago:Wago_734-132_1x02_P3.50mm_Vertical" H 1500 6800 50  0001 C CNN
+F 2 "TerminalBlock:TerminalBlock_bornier-2_P5.08mm" H 1500 6800 50  0001 C CNN
 F 3 "~" H 1500 6800 50  0001 C CNN
 	1    1500 6800
@@
 Wire Wire Line
 	3150 4500 3700 4500
+Wire Wire Line
+	3800 2050 3800 2500
+Wire Wire Line
+	3800 1600 3800 1750
+Wire Wire Line
+	3800 1750 4600 1750
+Wire Wire Line
+	4600 1750 4600 1600
 $EndSCHEMATC
